File: MEPOS_TEMPLATE/Base PCB.kicad_sch (KiCad schematic)
At the start: 8 parts, among them J201 Conn_02x32_Odd_Even, J202 Conn_02x20_Odd_Even

Commit message: Updated to MEPOS V0.5
-updated pinout so pin names matched schematic.
-added paste holes for alignment
Other:
- note added: "MEPOS Base PCB V22.04.0.5"
- note removed: "MEPOS Base PCB V22.04.0.4"
Changed lines of the file:
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@@
   (title_block
     (title "MEPOS Base PCB")
-    (date "2022-04-24")
-    (rev "V22.04.0.4")
+    (date "2022-05-15")
+    (rev "V22.04.0.5")
   )
   (junction (at 50.8 176.53) (diameter 0) (color 0 0 0 0)
@@
     (stroke (width 0) (type default) (color 0 0 0 0))
   )
-  (text "MEPOS Base PCB V22.04.0.4" (at 25.4 25.4 0)
+  (text "MEPOS Base PCB V22.04.0.5" (at 25.4 25.4 0)
     (effects (font (size 5.0038 5.0038) (thickness 1.0008) bold) (justify left bottom))
   )

Commit message: Updated Libraries
Parts:
- GND201: footprint MEP_TEMPLATE:Scope_GND -> MEPOS:Scope_GND
Changed lines of the file:
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@@
       (effects (font (size 1.27 1.27)) (justify left))
     )
-    (property "Footprint" "MEP_TEMPLATE:Scope_GND" (id 2) (at 31.75 165.1 0)
+    (property "Footprint" "MEPOS:Scope_GND" (id 2) (at 31.75 165.1 0)
       (effects (font (size 1.27 1.27)) hide)
     )

Commit message: Updated to MEPOS V22.07.0.51
Added fiducial markers to the topside of the board
Parts:
- added FID1, FID2, FID3, FID4: Fiducial, Fiducial:Fiducial_0.75mm_Mask1.5mm, symbol Mechanical:Fiducial
- GND1: renamed from GND201; now left out of the parts list
- H1: renamed from H201; now left out of the parts list
- H2: renamed from H202; now left out of the parts list
- H3: renamed from H203; now left out of the parts list
- H4: renamed from H204; now left out of the parts list
- renumbered J201 to J1, J202 to J2, JP201 to JP1
Other:
- note added: "MEPOS Base PCB V22.04.0.51"
- note removed: "MEPOS Base PCB V22.04.0.5"
Changed lines of the file:
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@@
   (title_block
     (title "MEPOS Base PCB")
-    (date "2022-05-15")
-    (rev "V22.04.0.5")
+    (date "2022-07-28")
+    (rev "V22.04.0.51")
   )
   (junction (at 50.8 176.53) (diameter 0) (color 0 0 0 0)
@@
     (stroke (width 0) (type default) (color 0 0 0 0))
   )
-  (text "MEPOS Base PCB V22.04.0.5" (at 25.4 25.4 0)
+  (text "MEPOS Base PCB V22.04.0.51" (at 25.4 25.4 0)
     (effects (font (size 5.0038 5.0038) (thickness 1.0008) bold) (justify left bottom))
   )
@@
   )
   (symbol (lib_id "Mechanical:MountingHole_Pad") (at 50.8 165.1 0) (unit 1)
-    (in_bom yes) (on_board yes)
-    (property "Reference" "H204" (id 0) (at 53.34 163.8554 0)
+    (in_bom no) (on_board yes)
+    (property "Reference" "H4" (id 0) (at 53.34 163.8554 0)
       (effects (font (size 1.27 1.27)) (justify left))
     )
@@
   )
   (symbol (lib_id "Mechanical:MountingHole_Pad") (at 31.75 165.1 0) (unit 1)
-    (in_bom yes) (on_board yes)
-    (property "Reference" "GND201" (id 0) (at 34.29 163.8554 0)
+    (in_bom no) (on_board yes)
+    (property "Reference" "GND1" (id 0) (at 34.29 163.8554 0)
       (effects (font (size 1.27 1.27)) (justify left))
     )
@@
   (symbol (lib_id "power:GND") (at 50.8 177.8 0) (unit 1)
     (in_bom yes) (on_board yes)
-    (property "Reference" "#PWR0201" (id 0) (at 50.8 184.15 0)
+    (property "Reference" "#PWR01" (id 0) (at 50.8 184.15 0)
       (effects (font (size 1.27 1.27)) hide)
     )
@@
   (symbol (lib_id "Device:Jumper_NO_Small") (at 50.8 172.72 270) (unit 1)
     (in_bom yes) (on_board yes)
-    (property "Reference" "JP201" (id 0) (at 52.0192 171.5516 90)
+    (property "Reference" "JP1" (id 0) (at 52.0192 171.5516 90)
       (effects (font (size 1.27 1.27)) (justify left))
     )
@@
   )
   (symbol (lib_id "Mechanical:MountingHole") (at 50.8 158.75 0) (unit 1)
-    (in_bom yes) (on_board yes)
-    (property "Reference" "H203" (id 0) (at 53.34 157.5816 0)
+    (in_bom no) (on_board yes)
+    (property "Reference" "H3" (id 0) (at 53.34 157.5816 0)
       (effects (font (size 1.27 1.27)) (justify left))
     )
@@
   )
   (symbol (lib_id "Mechanical:MountingHole") (at 50.8 153.67 0) (unit 1)
-    (in_bom yes) (on_board yes)
-    (property "Reference" "H202" (id 0) (at 53.34 152.5016 0)
+    (in_bom no) (on_board yes)
+    (property "Reference" "H2" (id 0) (at 53.34 152.5016 0)
       (effects (font (size 1.27 1.27)) (justify left))
     )
@@
   )
   (symbol (lib_id "Mechanical:MountingHole") (at 50.8 148.59 0) (unit 1)
-    (in_bom yes) (on_board yes)
-    (property "Reference" "H201" (id 0) (at 53.34 147.4216 0)
+    (in_bom no) (on_board yes)
+    (property "Reference" "H1" (id 0) (at 53.34 147.4216 0)
       (effects (font (size 1.27 1.27)) (justify left))
     )
@@
   (symbol (lib_id "Connector_Generic:Conn_02x32_Odd_Even") (at 90.17 88.9 0) (mirror y) (unit 1)
     (in_bom yes) (on_board yes)
-    (property "Reference" "J201" (id 0) (at 88.9 45.2882 0))
+    (property "Reference" "J1" (id 0) (at 88.9 45.2882 0))
     (property "Value" "Conn_02x32_Odd_Even" (id 1) (at 88.9 47.5996 0))
     (property "Footprint" "Connector_PinSocket_2.54mm:PinSocket_2x32_P2.54mm_Vertical" (id 2) (at 90.17 88.9 0)
@@
   (symbol (lib_id "Connector_Generic:Conn_02x20_Odd_Even") (at 204.47 86.36 0) (mirror y) (unit 1)
     (in_bom yes) (on_board yes)
-    (property "Reference" "J202" (id 0) (at 203.2 57.9882 0))
+    (property "Reference" "J2" (id 0) (at 203.2 57.9882 0))
     (property "Value" "Conn_02x20_Odd_Even" (id 1) (at 203.2 60.2996 0))
     (property "Footprint" "Connector_PinSocket_2.54mm:PinSocket_2x20_P2.54mm_Vertical" (id 2) (at 204.47 86.36 0)
@@
     (pin "9")
   )
+  (symbol (lib_id "Mechanical:Fiducial") (at 76.2 158.75 0) (unit 1)
+    (in_bom no) (on_board yes) (fields_autoplaced)
+    (property "Reference" "FID3" (id 0) (at 78.74 157.4799 0)
+      (effects (font (size 1.27 1.27)) (justify left))
+    )
+    (property "Value" "Fiducial" (id 1) (at 78.74 160.0199 0)
+      (effects (font (size 1.27 1.27)) (justify left))
+    )
+    (property "Footprint" "Fiducial:Fiducial_0.75mm_Mask1.5mm" (id 2) (at 76.2 158.75 0)
+      (effects (font (size 1.27 1.27)) hide)
+    )
+    (property "Datasheet" "~" (id 3) (at 76.2 158.75 0)
+      (effects (font (size 1.27 1.27)) hide)
+    )
+  )
+  (symbol (lib_id "Mechanical:Fiducial") (at 76.2 163.83 0) (unit 1)
+    (in_bom no) (on_board yes) (fields_autoplaced)
+    (property "Reference" "FID4" (id 0) (at 78.74 162.5599 0)
+      (effects (font (size 1.27 1.27)) (justify left))
+    )
+    (property "Value" "Fiducial" (id 1) (at 78.74 165.0999 0)
+      (effects (font (size 1.27 1.27)) (justify left))
+    )
+    (property "Footprint" "Fiducial:Fiducial_0.75mm_Mask1.5mm" (id 2) (at 76.2 163.83 0)
+      (effects (font (size 1.27 1.27)) hide)
+    )
+    (property "Datasheet" "~" (id 3) (at 76.2 163.83 0)
+      (effects (font (size 1.27 1.27)) hide)
+    )
+  )
+  (symbol (lib_id "Mechanical:Fiducial") (at 76.2 148.59 0) (unit 1)
+    (in_bom no) (on_board yes) (fields_autoplaced)
+    (property "Reference" "FID1" (id 0) (at 78.74 147.3199 0)
+      (effects (font (size 1.27 1.27)) (justify left))
+    )
+    (property "Value" "Fiducial" (id 1) (at 78.74 149.8599 0)
+      (effects (font (size 1.27 1.27)) (justify left))
+    )
+    (property "Footprint" "Fiducial:Fiducial_0.75mm_Mask1.5mm" (id 2) (at 76.2 148.59 0)
+      (effects (font (size 1.27 1.27)) hide)
+    )
+    (property "Datasheet" "~" (id 3) (at 76.2 148.59 0)
+      (effects (font (size 1.27 1.27)) hide)
+    )
+  )
+  (symbol (lib_id "Mechanical:Fiducial") (at 76.2 153.67 0) (unit 1)
+    (in_bom no) (on_board yes) (fields_autoplaced)
+    (property "Reference" "FID2" (id 0) (at 78.74 152.3999 0)
+      (effects (font (size 1.27 1.27)) (justify left))
+    )
+    (property "Value" "Fiducial" (id 1) (at 78.74 154.9399 0)
+      (effects (font (size 1.27 1.27)) (justify left))
+    )
+    (property "Footprint" "Fiducial:Fiducial_0.75mm_Mask1.5mm" (id 2) (at 76.2 153.67 0)
+      (effects (font (size 1.27 1.27)) hide)
+    )
+    (property "Datasheet" "~" (id 3) (at 76.2 153.67 0)
+      (effects (font (size 1.27 1.27)) hide)
+    )
+  )
 )
